File: V1_mcp2515_based/V1_mcp2515_based.kicad_sch (KiCad schematic)
At the start: 11 parts

Commit message: r
Parts:
- removed A?: (no value), symbol MCU_Module:Arduino_UNO_R3
- added A1: Arduino_UNO_R3, Module:Arduino_UNO_R3, symbol MCU_Module:Arduino_UNO_R3
- added R1: (no value), symbol Device:R_Small
- added R2, R3, R4: 4k7, Resistor_THT:R_Axial_DIN0204_L3.6mm_D1.6mm_P5.08mm_Horizontal, symbol Device:R_Small
- added U1: RP2040, MCU_RaspberryPi_and_Boards:RPi_Pico_SMD_TH, symbol MCU_RaspberryPi_RP2040:RP2040
- added U2: ESP32-S3-DevKitC, Espressif:ESP32-S3-DevKitC, symbol Espressif:ESP32-S3-DevKitC
- C1: renamed from C3; value (none) -> C_Small; footprint (none) -> Capacitor_THT:C_Disc_D4.7mm_W2.5mm_P5.00mm
- C2: renamed from C1; value (none) -> 100n; footprint (none) -> Capacitor_THT:C_Disc_D4.7mm_W2.5mm_P5.00mm
- C3: renamed from C2; value (none) -> 100n; footprint (none) -> Capacitor_THT:C_Disc_D4.7mm_W2.5mm_P5.00mm
- IC1: value (none) -> MCP2515-I_P; footprint (none) -> SamacSys_Parts:DIP794W56P254L2286H533Q18N
- J1: value (none) -> Screw_Terminal_01x03; footprint (none) -> TerminalBlock:TerminalBlock_Altech_AK300-3_P5.00mm
- JP1: value (none) -> Jumper_3_Open; footprint (none) -> Connector_PinHeader_2.54mm:PinHeader_1x03_P2.54mm_Vertical
- R5: renamed from R3; value (none) -> R_Small; footprint (none) -> Resistor_THT:R_Axial_DIN0204_L3.6mm_D1.6mm_P5.08mm_Horizontal
- R7: renamed from R2; value (none) -> 1-10k; footprint (none) -> Resistor_THT:R_Axial_DIN0204_L3.6mm_D1.6mm_P5.08mm_Horizontal
- Y1: value (none) -> Resonator_Small; footprint (none) -> Crystal:Resonator_Murata_CSTLSxxxG-3Pin_W8.0mm_H3.0mm
- renumbered R1 to R6
Connections:
- net +3V3: now also A1.4 (3V3), R1.1, R2.1, R3.1, R4.1, U1.36 (GPIO24), U2.1 (3V3), U2.2 (3V3)
- net +5V: now also A1.5 (+5V), U1.48 (USB_VDD), U2.21 (5V)
- net GND: now also A1.29 (GND), A1.6 (GND), A1.7 (GND), U1.57 (GND), U2.22 (GND), U2.23 (GND), U2.24 (GND), U2.44 (GND)
- net SPI_CLK: now also A1.13 (SDA/A4), R1.2, U2.20 (GPIO14/ADC2_CH3)
- net SPI_MISO: now also A1.12 (A3), R3.2, U2.18 (GPIO12/ADC2_CH1)
- net SPI_MOSI: now also A1.11 (A2), R2.2, U2.19 (GPIO13/ADC2_CH2)
- net SPI_SS: now also A1.10 (A1), R4.2, U2.8 (GPIO15/ADC2_CH4/32K_P)
- no-connect marks 0 -> 110
Other:
- note added: "ADJUSTABLE SPI PINS"
- note added: "FIXED SPI PINS"
- note added: "https://i0.wp.com/www.teachmemicro.com/wp-content/uploads/2021/12/Raspberry-Pi-Pico-Pinout.jpg?ssl=1"
- note added: "pull ups"
- moved on the sheet: C1, C2, C3, IC1, J1, JP1, R5, R6, R7, Y1

Commit message: h
Parts:
- removed C3: 100n, Capacitor_THT:C_Disc_D4.7mm_W2.5mm_P5.00mm, symbol Device:C_Small
- removed J1: Screw_Terminal_01x03, TerminalBlock:TerminalBlock_Altech_AK300-3_P5.00mm, symbol Connector:Screw_Terminal_01x03
- removed R2, R3: 4k7, Resistor_THT:R_Axial_DIN0204_L3.6mm_D1.6mm_P5.08mm_Horizontal, symbol Device:R_Small
- removed R7: 1-10k, Resistor_THT:R_Axial_DIN0204_L3.6mm_D1.6mm_P5.08mm_Horizontal, symbol Device:R_Small
- added C2: C_Small, Capacitor_THT:C_Disc_D4.3mm_W1.9mm_P5.00mm, symbol Device:C_Small
- added J1, J2: Screw_Terminal_01x02, TerminalBlock:TerminalBlock_Altech_AK300-2_P5.00mm, symbol Connector:Screw_Terminal_01x02
- added J3: (no value), symbol Connector_Generic:Conn_01x01
- added J4: Conn_01x07, Connector_PinHeader_2.54mm:PinHeader_1x07_P2.54mm_Vertical, symbol Connector_Generic:Conn_01x09
- added J5: SD_Card, symbol Connector:SD_Card
- added R4, R6: R_Small, Resistor_THT:R_Axial_DIN0204_L3.6mm_D1.6mm_P5.08mm_Horizontal, symbol Device:R_Small
- added U2: LF50_TO220, Package_TO_SOT_THT:TO-220-3_Vertical, symbol Regulator_Linear:LF50_TO220
- C1: footprint Capacitor_THT:C_Disc_D4.7mm_W2.5mm_P5.00mm -> Capacitor_THT:C_Disc_D4.3mm_W1.9mm_P5.00mm
- R1: value (none) -> 4k7; footprint (none) -> Resistor_THT:R_Axial_DIN0204_L3.6mm_D1.6mm_P5.08mm_Horizontal
- renumbered C2 to C3, R4 to R2, R6 to R3, U2 to U3
Connections:
- net +3V3: now also J4.4 (Pin_4), J5.4 (VDD), R6.1
- net +5V: now also C2.1, U2.3 (VO)
- net GND: now also C1.1, R5.1, C2.2, J1.2 (Pin_2), J4.3 (Pin_3), J4.6 (Pin_6), J5.3 (VSS), J5.6 (VSS), U2.2 (GND)
- net SPI_CLK: no longer R1.2
- net SPI_MISO: now also R4.2; no longer U3.18 (GPIO12/ADC2_CH1)
- net SPI_MISO_L: now reaches R5.2
- net SPI_MISO_L: now also U3.18 (GPIO12/ADC2_CH1), R4.1
- net +12V: now reaches C1.2
- net +12V: now also J1.1 (Pin_1), U2.1 (VI)
- net at IC1.1 (TXCAN): now also J2.1 (Pin_1)
- net at IC1.17 (~{RESET}): now also J3.1 (Pin_1)
- net at IC1.2 (RXCAN): now also J2.2 (Pin_2)
- new net CLK: J4.5 (Pin_5), J5.5 (CLK)
- new net MISO: J4.7 (Pin_7), J5.7 (DAT0)
- new net MOSI: J4.2 (Pin_2), J5.2 (CMD)
- new net SS: J4.1 (Pin_1), J5.1 (CD/DAT3), R1.2, R6.2
- no-connect marks 110 -> 113
