File: V1_mcp2515_based/V1_mcp2515_based.kicad_pcb (KiCad board)
At the start: 2 copper layers, 10 parts, among them IC1 MCP2515-I_P, J1 Screw_Terminal_01x03, Y1 Resonator_Small

Commit message: r
Parts:
- added A1: Arduino_UNO_R3, Module:Arduino_UNO_R3, F.Cu at (168.7, 65.5)
- added R1: 4k7, Resistor_THT:R_Axial_DIN0204_L3.6mm_D1.6mm_P5.08mm_Horizontal, F.Cu at (53.1, 72.9)
- added R2: 4k7, Resistor_THT:R_Axial_DIN0204_L3.6mm_D1.6mm_P5.08mm_Horizontal, F.Cu at (53.1, 69.8)
- added R3: 4k7, Resistor_THT:R_Axial_DIN0204_L3.6mm_D1.6mm_P5.08mm_Horizontal, F.Cu at (53.1, 67.1)
- added R4: 4k7, Resistor_THT:R_Axial_DIN0204_L3.6mm_D1.6mm_P5.08mm_Horizontal, F.Cu at (53.1, 63.8)
- added U1: RP2040, MCU_RaspberryPi_and_Boards:RPi_Pico_SMD_TH, F.Cu at (249.1, 88.8)
- added U2: ESP32-S3-DevKitC, Espressif:ESP32-S3-DevKitC, F.Cu at (212.1, 69.8)
- moved R6 79.8 mm to (27.7, 73.2)
- moved JP1 63.4 mm to (48.5, 54.9)
- moved J1 51.2 mm to (27.2, 52.9), turned to -90 degrees
- moved C2 45.3 mm to (44.4, 55.1), turned to 180 degrees
- moved Y1 37.5 mm to (32.5, 76.7), turned to 180 degrees
- moved C3 36.9 mm to (65.8, 132.8)
- moved IC1 28.6 mm to (40.4, 69.1)
- renumbered C3 to C1, C1 to C2, C2 to C3, R3 to R5, R1 to R6, R2 to R7

Commit message: h
Parts:
- removed the C3 at (65.8, 132.8)
- removed the R2 at (53.1, 69.8)
- removed the R3 at (53.1, 67.1)
- removed R7: 1-10k, Resistor_THT:R_Axial_DIN0204_L3.6mm_D1.6mm_P5.08mm_Horizontal
- added C2: C_Small, Capacitor_THT:C_Disc_D4.3mm_W1.9mm_P5.00mm, F.Cu at (45.3, 168.4)
- added J2: Screw_Terminal_01x02, TerminalBlock:TerminalBlock_Altech_AK300-2_P5.00mm, F.Cu at (134.1, 166.3)
- added J3: Conn_01x01, Connector_PinHeader_2.54mm:PinHeader_1x01_P2.54mm_Vertical, F.Cu at (113.0, 158.5)
- added J4: Conn_01x07, Connector_PinHeader_2.54mm:PinHeader_1x07_P2.54mm_Vertical, F.Cu at (130.0, 102.6)
- added R4: R_Small, Resistor_THT:R_Axial_DIN0204_L3.6mm_D1.6mm_P5.08mm_Horizontal, F.Cu at (122.9, 121.2)
- added R6: R_Small, Resistor_THT:R_Axial_DIN0204_L3.6mm_D1.6mm_P5.08mm_Horizontal, F.Cu at (131.0, 121.2)
- added U2: LF50_TO220, Package_TO_SOT_THT:TO-220-3_Vertical, F.Cu at (45.3, 159.0)
- C1: footprint Capacitor_THT:C_Disc_D4.7mm_W2.5mm_P5.00mm -> Capacitor_THT:C_Disc_D4.3mm_W1.9mm_P5.00mm
- J1: value Screw_Terminal_01x03 -> Screw_Terminal_01x02; footprint TerminalBlock:TerminalBlock_Altech_AK300-3_P5.00mm -> TerminalBlock:TerminalBlock_Altech_AK300-2_P5.00mm
- moved U1 177.9 mm to (77.0, 133.9), turned to 90 degrees
- moved C3 133.9 mm to (117.9, 167.1), turned to 0 degrees
- moved R3 130.5 mm to (134.4, 148.3), turned to 180 degrees
- moved JP1 129.7 mm to (113.0, 167.4), turned to 180 degrees
- moved Y1 118.7 mm to (129.6, 145.0), turned to 0 degrees
- moved IC1 117.3 mm to (121.9, 153.4), turned to 180 degrees
- moved U3 113.7 mm to (108.7, 116.8), turned to -90 degrees
- moved A1 111.7 mm to (67.1, 112.0)
- moved J1 106.5 mm to (35.8, 159.0)
- moved R2 100.2 mm to (127.5, 130.8)
- moved R1 93.3 mm to (131.0, 124.3), turned to 0 degrees
- moved R5 73.0 mm to (122.9, 124.3)
- moved C1 57.1 mm to (40.7, 154.2)
- renumbered C2 to C3, R4 to R2, R6 to R3, U2 to U3
Connections:
- C1 pad 1: unconnected-(C1-Pad1) -> GND
- C1 pad 2: unconnected-(C1-Pad2) -> +12V
- IC1 pad 17: unconnected-(IC1-Pad17) -> Net-(IC1-Pad17)
- J1 pad 1: GND -> +12V
- J1 pad 2: Net-(IC1-Pad1) -> GND
- R1 pad 2: SPI_CLK -> /SS
- R5 pad 1: unconnected-(R5-Pad1) -> GND
- R5 pad 2: unconnected-(R5-Pad2) -> SPI_MISO_L
- U3 pad 18: SPI_MISO -> SPI_MISO_L
Routing:
- added copper zone on B.Cu, net GND
Other:
- board outline added: 116.1 x 70.9 mm

Commit message: u
Connections:
- J2 pad 1: Net-(IC1-Pad2) -> Net-(IC1-Pad1)
- J2 pad 2: Net-(IC1-Pad1) -> Net-(IC1-Pad2)
Changed lines of the file:
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@@
     (fp_arc (start 3.39 -5) (mid 4.949737 -5.764867) (end 6.538239 -5.061686) (layer "F.Fab") (width 0.1))
     (pad "1" thru_hole rect (at 0 0 90) (size 1.98 3.96) (drill 1.32) (layers *.Cu *.Mask)
-      (net 6 "Net-(IC1-Pad2)") (pinfunction "Pin_1") (pintype "passive"))
+      (net 5 "Net-(IC1-Pad1)") (pinfunction "Pin_1") (pintype "passive"))
     (pad "2" thru_hole oval (at 5 0 90) (size 1.98 3.96) (drill 1.32) (layers *.Cu *.Mask)
-      (net 5 "Net-(IC1-Pad1)") (pinfunction "Pin_2") (pintype "passive"))
+      (net 6 "Net-(IC1-Pad2)") (pinfunction "Pin_2") (pintype "passive"))
     (model "${KICAD6_3DMODEL_DIR}/TerminalBlock.3dshapes/TerminalBlock_Altech_AK300-2_P5.00mm.wrl"
       (offset (xyz 0 0 0))
@@
     (connect_pads (clearance 0.508))
     (min_thickness 0.4) (filled_areas_thickness no)
-    (fill (thermal_gap 0.4) (thermal_bridge_width 0.7))
+    (fill yes (thermal_gap 0.4) (thermal_bridge_width 0.7))
     (polygon
       (pts
