File: V1_mcp2561_based/V1_mcp2561_based.kicad_sch (KiCad schematic)
At the start: 6 parts

Commit message: r
Parts:
- added C2: 4.7n, Capacitor_THT:C_Disc_D4.3mm_W1.9mm_P5.00mm, symbol Device:C_Small
- added R1: 300 optional, Resistor_THT:R_Axial_DIN0204_L3.6mm_D1.6mm_P5.08mm_Horizontal, symbol Device:R_Small
- added R2, R3: 60, Resistor_THT:R_Axial_DIN0204_L3.6mm_D1.6mm_P5.08mm_Horizontal, symbol Device:R_Small
- added U1: RP2040, MCU_RaspberryPi_and_Boards:RPi_Pico_SMD_TH, symbol MCU_RaspberryPi_RP2040:RP2040
- added U3: ESP32-S3-DevKitC, Espressif:ESP32-S3-DevKitC, symbol Espressif:ESP32-S3-DevKitC
- A1: value (none) -> Arduino_UNO_R3; footprint (none) -> Module:Arduino_UNO_R3
- C1: value C_Small -> 100n
- C3: renamed from C2; value (none) -> C_Small; footprint (none) -> Capacitor_THT:C_Disc_D4.3mm_W1.9mm_P5.00mm
- J1: value (none) -> Screw_Terminal_01x03; footprint (none) -> TerminalBlock:TerminalBlock_Altech_AK300-3_P5.00mm
- R4: renamed from R1; value (none) -> R_Small; footprint (none) -> Resistor_THT:R_Axial_DIN0204_L3.6mm_D1.6mm_P5.08mm_Horizontal
- U2: renamed from U1; value (none) -> MCP2561-E-P; footprint (none) -> Package_DIP:DIP-8_W7.62mm
Connections:
- net +5V: now also U1.48 (USB_VDD), U3.21 (5V)
- net GND: now also C2.2, U1.57 (GND), U3.22 (GND), U3.23 (GND), U3.24 (GND), U3.44 (GND)
- net +3V3: now reaches A1.4 (3V3)
- net +3V3: now also U1.36 (GPIO24), U3.1 (3V3), U3.2 (3V3)
- net SPL: now reaches U2.5 (SPLIT)
- net SPL: now also R1.2
- net CANH: now reaches J1.3 (Pin_3)
- net CANH: now also U2.7 (CANH), R2.1; no longer U2.6 (CANL)
- net CANL: now reaches J1.1 (Pin_1)
- net CANL: now also U2.6 (CANL), R3.2; no longer U2.7 (CANH)
- new net: C2.1, R1.1, R2.2, R3.1
- no-connect marks 0 -> 118
Other:
- note added: "OPTIONAL BUT NEEDED FOR EMC/EMI COOMON MODE CHOKE"
- note added: "only needed for data rates over 1Mbps in the case of cars data rtes are under or at that speed"
- moved on the sheet: A1, C1, C3, J1, R4, U2

Commit message: e
Parts:
- removed C3: C_Small, Capacitor_THT:C_Disc_D4.3mm_W1.9mm_P5.00mm, symbol Device:C_Small
- removed J1: Screw_Terminal_01x03, TerminalBlock:TerminalBlock_Altech_AK300-3_P5.00mm, symbol Connector:Screw_Terminal_01x03
- removed U1: RP2040, MCU_RaspberryPi_and_Boards:RPi_Pico_SMD_TH, symbol MCU_RaspberryPi_RP2040:RP2040
- added C1, C2: C_Small, Capacitor_THT:C_Disc_D4.3mm_W1.9mm_P5.00mm, symbol Device:C_Small
- added J1: (no value), symbol Connector:Screw_Terminal_01x02
- added J2: Screw_Terminal_01x02, TerminalBlock:TerminalBlock_Altech_AK300-2_P5.00mm, symbol Connector:Screw_Terminal_01x02
- added JP1: (no value), symbol Jumper:Jumper_2_Bridged
- added R1, R2: R_Small, Resistor_THT:R_Axial_DIN0204_L3.6mm_D1.6mm_P5.08mm_Horizontal, symbol Device:R_Small
- added R3: (no value), symbol Device:R_Small
- added U1: (no value), symbol Regulator_Linear:LF50_TO220
- added U2: (no value), symbol MCU_RaspberryPi_and_Boards:RP2040
- U3: renamed from U2; value MCP2561-E-P -> (none); footprint Package_DIP:DIP-8_W7.62mm -> (none)
- renumbered C1 to C3, C2 to C4, R1 to R5, R2 to R6, R3 to R7, U3 to U4
Connections:
- net +5V: now also C2.1, R3.2, U1.3 (VO), U2.40 (GPIO28_ADC2)
- net CANH: now also J1.2 (Pin_2)
- net CANL: now also J1.1 (Pin_1)
- net GND: now also C1.1, C2.2, J2.2 (Pin_2), JP1.1 (A), R2.2, U1.2 (GND), U2.1 (IOVDD)
- net STBY: now reaches A1.24 (D9)
- net STBY: now also U3.8 (STBY), U4.34 (GPIO37), JP1.2 (B), R3.1, U2.11 (GPIO8)
- net TX-pin: now reaches A1.26 (D11)
- net TX-pin: now also R4.1, U4.29 (GPIO48), U2.6 (GPIO4)
- net RXD: now reaches A1.27 (D12)
- net RXD: now also U3.4 (RXD), R1.1
- net TXD: now reaches U3.1 (TXD)
- net TXD: now also R4.2
- net RX-pin: now reaches U4.28 (GPIO47)
- net RX-pin: now also R1.2, R2.1, U2.5 (GPIO3)
- new net +12V: C1.2, J2.1 (Pin_1), U1.1 (VI)
- no-connect marks 118 -> 110
Other:
- note added: "3V3 TTL FOM 5V TTL"
- note added: "Max source sink current arduino ESP32 STM32 rp2040"
- note added: "just curent limiter"
- note added: "modes: STBY PIN: LOW bus is dominant ; wake up call is detected HIGH bus is recesive ; no wake up call deteted MY OPINION: set it LOW"
- moved on the sheet: U4

Commit message: h
Parts:
- added J2: (no value), symbol Connector_Generic:Conn_01x09
- added J4: (no value), symbol Connector:SD_Card
- added R1, R11, R2, R3, R4, R5, R6: R_Small, Resistor_THT:R_Axial_DIN0204_L3.6mm_D1.6mm_P5.08mm_Horizontal, symbol Device:R_Small
- renumbered C3 to C1, C1 to C2, C2 to C3, J2 to J3, R3 to R10, R5 to R12, R6 to R13, R7 to R14, R1 to R7, R2 to R8, R4 to R9, U4 to U1, U1 to U4
Connections:
- net +3V3: now also U1.17 (GPIO11/ADC2_CH0), U2.36 (GPIO24), J2.4 (Pin_4), J4.4 (VDD), R11.1
- net GND: now also J2.3 (Pin_3), J2.6 (Pin_6), J4.3 (VSS), J4.6 (VSS), R2.2, R4.2, R6.2
- net at A1.10 (A1): now also R5.1
- net at A1.11 (A2): now also R3.1
- net MISO: now reaches A1.12 (A3)
- net MISO: now also U1.4 (GPIO4/ADC1_CH3), J2.7 (Pin_7), J4.7 (DAT0)
- net at A1.13 (SDA/A4): now also R1.1
- net SS: now reaches U1.5 (GPIO5/ADC1_CH4)
- net SS: now also J2.1 (Pin_1), J4.1 (CD/DAT3), R11.2, R5.2, R6.1
- net MOSI: now reaches U1.6 (GPIO6/ADC1_CH5)
- net MOSI: now also J2.2 (Pin_2), J4.2 (CMD), R3.2, R4.1
- net CLK: now reaches U1.8 (GPIO15/ADC2_CH4/32K_P)
- net CLK: now also J2.5 (Pin_5), J4.5 (CLK), R1.2, R2.1
- no-connect marks 110 -> 107
Other:
- note added: "Max source sink current arduino 8 8mA ESP32 40 28mA STM32 25 25mA rp2040"
- note removed: "Max source sink current arduino ESP32 STM32 rp2040"
- moved on the sheet: A1, C1, C2, C3, C4, J1, J3, JP1, R10, R12, R13, R14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
