File: V1_mini_mcp2515_based/V1_mini_mcp2515_based.kicad_sch (KiCad schematic)
At the start: 20 parts, among them IC1 MCP2515-I_P, J1 Conn_01x07, J2 Screw_Terminal_01x02, J3 SD_Card, J4 Conn_01x01, J6 Conn_01x05, J7 Conn_01x05, J8 Screw_Terminal_01x02, Y1 Resonator_Small

Commit message: f
Parts:
- removed J6: Conn_01x05, Connector_PinHeader_2.54mm:PinHeader_1x05_P2.54mm_Vertical, symbol Connector_Generic:Conn_01x05
- added J10, J11, J3: Conn_01x01, Connector_PinHeader_2.54mm:PinHeader_1x01_P2.54mm_Vertical, symbol Connector_Generic:Conn_01x01
- added J14: (no value), symbol Connector_Generic:Conn_01x06
- added J4: (no value), symbol Connector_Generic:Conn_01x03
- added J6: Conn_01x03, Connector_PinHeader_2.54mm:PinHeader_1x03_P2.54mm_Vertical, symbol Connector_Generic:Conn_01x03
- added J8: (no value), Connector_PinHeader_2.54mm:PinHeader_1x03_P2.54mm_Vertical, symbol Connector_Generic:Conn_01x03
- added JP1: (no value), symbol Jumper:Jumper_2_Open
- added R10, R11, R12, R7, R8, R9: R_Small, Resistor_THT:R_Axial_DIN0204_L3.6mm_D1.6mm_P5.08mm_Horizontal, symbol Device:R_Small
- J1: value Conn_01x07 -> (none)
- J13: renamed from J7; value Conn_01x05 -> (none)
- J9: renamed from J5; footprint (none) -> Connector_PinHeader_2.54mm:PinHeader_1x05_P2.54mm_Vertical
- R2: value R_Small -> (none); footprint Resistor_THT:R_Axial_DIN0204_L3.6mm_D1.6mm_P5.08mm_Horizontal -> (none)
- U1: value (none) -> LF50_TO220; footprint (none) -> Package_TO_SOT_THT:TO-220-3_Horizontal_TabDown
- renumbered J8 to J12, J3 to J5, J4 to J7, R5 to R3, R6 to R4, R3 to R5, R4 to R6
Connections:
- net MOSI is gone; now on net SPI_MOSI: J1.2 (Pin_2), J13.4 (Pin_4), J5.2 (CMD)
- net +3V3: now also J10.1 (Pin_1), J11.1 (Pin_1), J8.1 (Pin_1)
- net +5V: now also J8.3 (Pin_3)
- net GND: now also J14.1 (Pin_1), J8.2 (Pin_2), JP1.1 (A); no longer R6.1
- net SPI_CLK: now also J1.5 (Pin_5), J13.3 (Pin_3), J5.5 (CLK), R5.2
- net SPI_MISO: now also J1.7 (Pin_7), J13.2 (Pin_2), J5.7 (DAT0), J14.3 (Pin_3)
- net SPI_MOSI: now also R7.2
- net SPI_SS: now also R9.2
- net SS: now also R11.2
- net at IC1.10 (~{RX1BF}): now also J6.3 (Pin_3)
- net at IC1.11 (~{RX0BF}): now also J6.2 (Pin_2)
- net at IC1.12 (~{INT}): now also J6.1 (Pin_1)
- net at IC1.3 (CLKOUT/SOF): now also J3.1 (Pin_1)
- net at IC1.4 (~{TX0RTS}): now also J4.1 (Pin_1)
- net at IC1.5 (~{TX1RTS}): now also J4.2 (Pin_2)
- net at IC1.6 (~{TX2RTS}): now also J4.3 (Pin_3)
- net at R5.1, R6.2: now also J14.2 (Pin_2)
- removed net CLK: J1.5 (Pin_5), J13.2 (Pin_2), J5.5 (CLK)
- removed net MISO: J1.7 (Pin_7), J13.3 (Pin_3), J5.7 (DAT0)
- new net: JP1.2 (B), R10.1, R12.1, R6.1, R8.1
- new net: J14.6 (Pin_6), R10.2, R9.1
- new net: J14.4 (Pin_4), R7.1, R8.2
- new net: J14.5 (Pin_5), R11.1, R12.2
- no-connect marks 3 -> 8
Other:
- note added: "TTL 3v3"
- note added: "TTL 5V/3v3"
- moved on the sheet: C2, C3, J12, J13, J2, J9, R1, R5, R6, U1, Y1

Commit message: t
Parts:
- IC1: footprint SamacSys_Parts:DIP794W56P254L2286H533Q18N -> Package_DIP:DIP-18_W7.62mm_LongPads
- J1: value (none) -> SD_crd
- J13: value (none) -> SPI2
- J14: value (none) -> SPI_AVR; footprint (none) -> Connector_PinHeader_2.54mm:PinHeader_1x06_P2.54mm_Vertical
- J4: value (none) -> Conn_01x03; footprint (none) -> Connector_PinHeader_2.54mm:PinHeader_1x03_P2.54mm_Vertical
- J8: value (none) -> power
- J9: value (none) -> SPI1
- JP1: value (none) -> Jumper_2_Open; footprint (none) -> Connector_PinHeader_2.54mm:PinHeader_1x02_P2.54mm_Vertical
- R2: value (none) -> 10k; footprint (none) -> Resistor_THT:R_Axial_DIN0204_L3.6mm_D1.6mm_P5.08mm_Horizontal
Changed lines of the file:
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@@
     (in_bom yes) (on_board yes)
     (property "Reference" "JP1" (id 0) (at 223.52 153.67 0))
-    (property "Value" "" (id 1) (at 223.52 156.21 0))
-    (property "Footprint" "" (id 2) (at 223.52 150.495 0)
+    (property "Value" "Jumper_2_Open" (id 1) (at 223.52 156.21 0))
+    (property "Footprint" "Connector_PinHeader_2.54mm:PinHeader_1x02_P2.54mm_Vertical" (id 2) (at 223.52 150.495 0)
       (effects (font (size 1.27 1.27)) hide)
     )
@@
     (in_bom yes) (on_board yes) (fields_autoplaced)
     (property "Reference" "J14" (id 0) (at 215.9 107.95 0))
-    (property "Value" "" (id 1) (at 215.9 110.49 0))
-    (property "Footprint" "" (id 2) (at 215.9 122.555 0)
+    (property "Value" "SPI_AVR" (id 1) (at 215.9 110.49 0))
+    (property "Footprint" "Connector_PinHeader_2.54mm:PinHeader_1x06_P2.54mm_Vertical" (id 2) (at 215.9 122.555 0)
       (effects (font (size 1.27 1.27)) hide)
     )
@@
     (in_bom yes) (on_board yes) (fields_autoplaced)
     (property "Reference" "J9" (id 0) (at 154.305 109.855 0))
-    (property "Value" "" (id 1) (at 154.305 112.395 0))
+    (property "Value" "SPI1" (id 1) (at 154.305 112.395 0))
     (property "Footprint" "Connector_PinHeader_2.54mm:PinHeader_1x05_P2.54mm_Vertical" (id 2) (at 154.305 121.92 0)
       (effects (font (size 1.27 1.27)) hide)
@@
     (property "Reference" "IC1" (id 0) (at 93.98 33.02 0))
     (property "Value" "MCP2515-I_P" (id 1) (at 93.98 35.56 0))
-    (property "Footprint" "SamacSys_Parts:DIP794W56P254L2286H533Q18N" (id 2) (at 109.22 38.1 0)
+    (property "Footprint" "Package_DIP:DIP-18_W7.62mm_LongPads" (id 2) (at 109.22 38.1 0)
       (effects (font (size 1.27 1.27)) (justify left) hide)
     )
@@
     (in_bom yes) (on_board yes) (fields_autoplaced)
     (property "Reference" "R2" (id 0) (at 59.69 105.41 90))
-    (property "Value" "" (id 1) (at 59.69 107.95 90))
-    (property "Footprint" "" (id 2) (at 59.69 111.76 0)
+    (property "Value" "10k" (id 1) (at 59.69 107.95 90))
+    (property "Footprint" "Resistor_THT:R_Axial_DIN0204_L3.6mm_D1.6mm_P5.08mm_Horizontal" (id 2) (at 59.69 111.76 0)
       (effects (font (size 1.27 1.27)) hide)
     )
@@
     (in_bom yes) (on_board yes) (fields_autoplaced)
     (property "Reference" "J13" (id 0) (at 191.135 109.855 0))
-    (property "Value" "" (id 1) (at 191.135 112.395 0))
+    (property "Value" "SPI2" (id 1) (at 191.135 112.395 0))
     (property "Footprint" "Connector_PinHeader_2.54mm:PinHeader_1x05_P2.54mm_Vertical" (id 2) (at 191.135 121.92 0)
       (effects (font (size 1.27 1.27)) hide)
@@
     (in_bom yes) (on_board yes)
     (property "Reference" "J4" (id 0) (at 59.055 50.8 0))
-    (property "Value" "" (id 1) (at 59.055 53.34 0))
-    (property "Footprint" "" (id 2) (at 66.675 50.8 0)
+    (property "Value" "Conn_01x03" (id 1) (at 59.055 53.34 0))
+    (property "Footprint" "Connector_PinHeader_2.54mm:PinHeader_1x03_P2.54mm_Vertical" (id 2) (at 66.675 50.8 0)
       (effects (font (size 1.27 1.27)) hide)
     )
@@
     (in_bom yes) (on_board yes)
     (property "Reference" "J8" (id 0) (at 141.605 83.185 0))
-    (property "Value" "" (id 1) (at 141.605 80.645 0))
+    (property "Value" "power" (id 1) (at 141.605 80.645 0))
     (property "Footprint" "Connector_PinHeader_2.54mm:PinHeader_1x03_P2.54mm_Vertical" (id 2) (at 149.225 81.28 0)
       (effects (font (size 1.27 1.27)) hide)
@@
     (in_bom yes) (on_board yes) (fields_autoplaced)
     (property "Reference" "J1" (id 0) (at 36.195 110.49 0))
-    (property "Value" "" (id 1) (at 36.195 113.03 0))
+    (property "Value" "SD_crd" (id 1) (at 36.195 113.03 0))
     (property "Footprint" "Connector_PinHeader_2.54mm:PinHeader_1x07_P2.54mm_Vertical" (id 2) (at 36.195 127.635 0)
       (effects (font (size 1.27 1.27)) hide)
@@
     )
     (path "/560d05a7-84e4-403a-80d1-f287a4032b8a"
-      (reference "IC1") (unit 1) (value "MCP2515-I_P") (footprint "SamacSys_Parts:DIP794W56P254L2286H533Q18N")
+      (reference "IC1") (unit 1) (value "MCP2515-I_P") (footprint "Package_DIP:DIP-18_W7.62mm_LongPads")
     )
     (path "/cd8b6ef6-f2d8-48ae-bd83-6d4627d39e9b"
